File: MegaCD Cable Adapter.kicad_sch (KiCad schematic)
At the start: 8 parts, among them J1 Mega CD Edge Connector, J1 Mega CD Header

Commit message: Work on v2
Parts:
- C1, C2: footprint Capacitor_THT:CP_Radial_D5.0mm_P2.50mm -> (none)
- D1, D2: footprint LED_THT:LED_D3.0mm -> (none)
- J1: footprint Sega:PinHeader_2x30_P2.54mm_Vertical_AB_Numbering -> (none)
- R1, R2: footprint Resistor_THT:R_Axial_DIN0207_L6.3mm_D2.5mm_P10.16mm_Horizontal -> Resistor_SMD:R_1206_3216Metric_Pad1.30x1.75mm_HandSolder
Changed lines of the file:
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@@
       (effects (font (size 1.27 1.27)) (justify left))
     )
-    (property "Footprint" "Capacitor_THT:CP_Radial_D5.0mm_P2.50mm" (at 228.6 30.48 0)
+    (property "Footprint" "" (at 228.6 30.48 0)
       (effects (font (size 1.27 1.27)) hide)
     )
@@
       (effects (font (size 1.27 1.27)))
     )
-    (property "Footprint" "Resistor_THT:R_Axial_DIN0207_L6.3mm_D2.5mm_P10.16mm_Horizontal" (at 236.474 90.424 90)
+    (property "Footprint" "Resistor_SMD:R_1206_3216Metric_Pad1.30x1.75mm_HandSolder" (at 236.474 90.424 90)
       (effects (font (size 1.27 1.27)) hide)
     )
@@
       (effects (font (size 1.27 1.27)))
     )
-    (property "Footprint" "LED_THT:LED_D3.0mm" (at 223.52 91.44 0)
+    (property "Footprint" "" (at 223.52 91.44 0)
       (effects (font (size 1.27 1.27)) hide)
     )
@@
       (effects (font (size 1.27 1.27)) (justify left))
     )
-    (property "Footprint" "Capacitor_THT:CP_Radial_D5.0mm_P2.50mm" (at 229.5652 59.69 0)
+    (property "Footprint" "" (at 229.5652 59.69 0)
       (effects (font (size 1.27 1.27)) hide)
     )
@@
       (effects (font (size 1.27 1.27)))
     )
-    (property "Footprint" "LED_THT:LED_D3.0mm" (at 223.52 104.14 0)
+    (property "Footprint" "" (at 223.52 104.14 0)
       (effects (font (size 1.27 1.27)) hide)
     )
@@
       (effects (font (size 1.27 1.27)))
     )
-    (property "Footprint" "Sega:PinHeader_2x30_P2.54mm_Vertical_AB_Numbering" (at 53.34 58.42 0)
+    (property "Footprint" "" (at 53.34 58.42 0)
       (effects (font (size 1.27 1.27)) hide)
     )
@@
       (effects (font (size 1.27 1.27)))
     )
-    (property "Footprint" "Resistor_THT:R_Axial_DIN0207_L6.3mm_D2.5mm_P10.16mm_Horizontal" (at 236.474 103.124 90)
-      (effects (font (size 1.27 1.27)) hide)
-    )
+    (property "Footprint" "Resistor_SMD:R_1206_3216Metric_Pad1.30x1.75mm_HandSolder" (at 236.474 103.124 90)
+      (effects (font (size 1.27 1.27)) hide)
+    )
