File: Teradrive Mega CD Adapter.kicad_pcb (KiCad board)
At the start: 2 copper layers, 63.8 x 87.4 mm, 77 parts, among them J1 Mega CD Header, J2 Tera Drive Expansion Port

Commit message: Work on v2
Parts:
- removed C1, C2: 47μF, Capacitor_THT:CP_Radial_D5.0mm_P2.50mm
- removed D1: +5V Indicator, LED_THT:LED_D3.0mm
- removed D2: +9V Indicator, LED_THT:LED_D3.0mm
- removed JPA1, JPA11, JPA12, JPA13, JPA14, JPA15, JPA16, JPA17, JPA22, JPA23, JPA24, JPA25, JPA26, JPA27, JPA28, JPA29, JPA3, JPA32, JPA4, JPA5, JPA6, JPB1, JPB10, JPB11, JPB12, JPB13, JPB14, JPB15, JPB16, JPB17, JPB18, JPB19, JPB20, JPB21, JPB22, JPB23, JPB24, JPB25, JPB26, JPB27, JPB28, JPB29, JPB3, JPB30, JPB32, JPB4, JPB5, JPB6, JPB7, JPB8, JPB9: SolderJumper_2_Open, Sega:SolderJumper-2_P1.3mm_Open_RoundedPad1.0x1.5mm_PretendShorted
- removed JPA31: Exp/Cart Boot, Connector_PinHeader_2.54mm:PinHeader_1x03_P2.54mm_Vertical
- removed JPB2: Sound 1 Left/Right, Connector_PinHeader_2.54mm:PinHeader_1x03_P2.54mm_Vertical
- removed JPB31: Sound 2 Left/Right, Connector_PinHeader_2.54mm:PinHeader_1x03_P2.54mm_Vertical
- removed TP9V1: MegaCD +9V, TestPoint:TestPoint_Pad_D1.5mm
- removed TPA10: Tera Drive extra address A_{23}, TestPoint:TestPoint_Pad_D1.5mm
- removed TPA18: Tera Drive cartridge chip enable (cart slot B17), TestPoint:TestPoint_Pad_D1.5mm
- removed TPA19: Tera Drive cartridge address strobe (cart slot B18), TestPoint:TestPoint_Pad_D1.5mm
- removed TPA2: Tera Drive cartridge reset (cart slot B2), TestPoint:TestPoint_Pad_D1.5mm
- removed TPA20: Tera Drive cartridge 68K data clock (cart slot B19), TestPoint:TestPoint_Pad_D1.5mm
- removed TPA21: Tera Drive cartridge data xfer ack (cart slot B20), TestPoint:TestPoint_Pad_D1.5mm
- removed TPA30: Tera Drive cartridge ??? signal (cart slot B31), TestPoint:TestPoint_Pad_D1.5mm
- removed TPA7: Tera Drive extra address A_{20}, TestPoint:TestPoint_Pad_D1.5mm
- removed TPA8: Tera Drive extra address A_{21}, TestPoint:TestPoint_Pad_D1.5mm
- removed TPA9: Tera Drive extra address A_{22}, TestPoint:TestPoint_Pad_D1.5mm
- removed TPSL3: MegaCD Sound Left 3 (unused), TestPoint:TestPoint_Pad_D1.5mm
- removed TPSR3: MegaCD Sound Right 3 (unused), TestPoint:TestPoint_Pad_D1.5mm
- added J5: Tera Drive Expansion Port, Sega:TE_1761469-1_BA_Numbering, B.Cu at (76.7, 105.8)
- added JP1: Exp/Cart Boot, Connector_PinHeader_2.54mm:PinHeader_1x03_P2.54mm_Vertical, F.Cu at (196.5, 147.6)
- added R10: 100Ω, Resistor_SMD:R_1206_3216Metric_Pad1.30x1.75mm_HandSolder, F.Cu at (125.0, 77.5)
- added R11: 100Ω, Resistor_SMD:R_1206_3216Metric_Pad1.30x1.75mm_HandSolder, F.Cu at (130.0, 77.5)
- added R12: 100Ω, Resistor_SMD:R_1206_3216Metric_Pad1.30x1.75mm_HandSolder, F.Cu at (127.5, 83.1)
- added R13: 100Ω, Resistor_SMD:R_1206_3216Metric_Pad1.30x1.75mm_HandSolder, F.Cu at (122.4, 83.1)
- added R14: 100Ω, Resistor_SMD:R_1206_3216Metric_Pad1.30x1.75mm_HandSolder, F.Cu at (117.3, 83.1)
- added R15: 100Ω, Resistor_SMD:R_1206_3216Metric_Pad1.30x1.75mm_HandSolder, F.Cu at (112.3, 83.1)
- added R16: 100Ω, Resistor_SMD:R_1206_3216Metric_Pad1.30x1.75mm_HandSolder, F.Cu at (107.2, 83.1)
- added R17: 100Ω, Resistor_SMD:R_1206_3216Metric_Pad1.30x1.75mm_HandSolder, F.Cu at (101.9, 83.1)
- added R18: 100Ω, Resistor_SMD:R_1206_3216Metric_Pad1.30x1.75mm_HandSolder, F.Cu at (97.0, 83.1)
- added R19: 100Ω, Resistor_SMD:R_1206_3216Metric_Pad1.30x1.75mm_HandSolder, F.Cu at (91.9, 83.1)
- added R20: 100Ω, Resistor_SMD:R_1206_3216Metric_Pad1.30x1.75mm_HandSolder, F.Cu at (240.4, 85.7)
- added R21: 100Ω, Resistor_SMD:R_1206_3216Metric_Pad1.30x1.75mm_HandSolder, F.Cu at (240.4, 89.0)
- added R22: 100Ω, Resistor_SMD:R_1206_3216Metric_Pad1.30x1.75mm_HandSolder, F.Cu at (240.4, 92.3)
- added R23: 100Ω, Resistor_SMD:R_1206_3216Metric_Pad1.30x1.75mm_HandSolder, F.Cu at (246.3, 66.0)
- added R24: 100Ω, Resistor_SMD:R_1206_3216Metric_Pad1.30x1.75mm_HandSolder, F.Cu at (246.3, 69.3)
- added R25: 100Ω, Resistor_SMD:R_1206_3216Metric_Pad1.30x1.75mm_HandSolder, F.Cu at (246.3, 72.6)
- added R26: 100Ω, Resistor_SMD:R_1206_3216Metric_Pad1.30x1.75mm_HandSolder, F.Cu at (246.3, 75.9)
- added R27: 100Ω, Resistor_SMD:R_1206_3216Metric_Pad1.30x1.75mm_HandSolder, F.Cu at (246.3, 79.2)
- added R28: 100Ω, Resistor_SMD:R_1206_3216Metric_Pad1.30x1.75mm_HandSolder, F.Cu at (246.3, 82.4)
- added R29: 100Ω, Resistor_SMD:R_1206_3216Metric_Pad1.30x1.75mm_HandSolder, F.Cu at (246.3, 85.7)
- added R30: 100Ω, Resistor_SMD:R_1206_3216Metric_Pad1.30x1.75mm_HandSolder, F.Cu at (246.3, 89.0)
- added R31: 100Ω, Resistor_SMD:R_1206_3216Metric_Pad1.30x1.75mm_HandSolder, F.Cu at (246.3, 92.3)
- added R32: 100Ω, Resistor_SMD:R_1206_3216Metric_Pad1.30x1.75mm_HandSolder, F.Cu at (252.3, 66.0)
- added R33: 100Ω, Resistor_SMD:R_1206_3216Metric_Pad1.30x1.75mm_HandSolder, F.Cu at (252.3, 69.3)
- added R34: 100Ω, Resistor_SMD:R_1206_3216Metric_Pad1.30x1.75mm_HandSolder, F.Cu at (252.3, 72.6)
- added R35: 100Ω, Resistor_SMD:R_1206_3216Metric_Pad1.30x1.75mm_HandSolder, F.Cu at (252.3, 75.9)
- added R36: 100Ω, Resistor_SMD:R_1206_3216Metric_Pad1.30x1.75mm_HandSolder, F.Cu at (252.3, 79.2)
- added R37: 100Ω, Resistor_SMD:R_1206_3216Metric_Pad1.30x1.75mm_HandSolder, F.Cu at (252.3, 82.4)
- added R38: 100Ω, Resistor_SMD:R_1206_3216Metric_Pad1.30x1.75mm_HandSolder, F.Cu at (252.3, 85.7)
- added R39: 100Ω, Resistor_SMD:R_1206_3216Metric_Pad1.30x1.75mm_HandSolder, F.Cu at (252.3, 89.0)
- added R40: 100Ω, Resistor_SMD:R_1206_3216Metric_Pad1.30x1.75mm_HandSolder, F.Cu at (252.3, 92.3)
- added R41: 100Ω, Resistor_SMD:R_1206_3216Metric_Pad1.30x1.75mm_HandSolder, F.Cu at (258.2, 66.0)
- added R42: 100Ω, Resistor_SMD:R_1206_3216Metric_Pad1.30x1.75mm_HandSolder, F.Cu at (258.2, 69.3)
- added R43: 100Ω, Resistor_SMD:R_1206_3216Metric_Pad1.30x1.75mm_HandSolder, F.Cu at (258.2, 72.6)
- added R44: 100Ω, Resistor_SMD:R_1206_3216Metric_Pad1.30x1.75mm_HandSolder, F.Cu at (258.2, 75.9)
- added R45: 100Ω, Resistor_SMD:R_1206_3216Metric_Pad1.30x1.75mm_HandSolder, F.Cu at (258.2, 79.2)
- added R46: 100Ω, Resistor_SMD:R_1206_3216Metric_Pad1.30x1.75mm_HandSolder, F.Cu at (258.2, 82.4)
- added R5: 100Ω, Resistor_SMD:R_1206_3216Metric_Pad1.30x1.75mm_HandSolder, F.Cu at (99.6, 77.7)
- added R6: 100Ω, Resistor_SMD:R_1206_3216Metric_Pad1.30x1.75mm_HandSolder, F.Cu at (104.6, 77.7)
- added R7: 100Ω, Resistor_SMD:R_1206_3216Metric_Pad1.30x1.75mm_HandSolder, F.Cu at (109.7, 77.5)
- added R8: 100Ω, Resistor_SMD:R_1206_3216Metric_Pad1.30x1.75mm_HandSolder, F.Cu at (114.8, 77.5)
- added R9: 100Ω, Resistor_SMD:R_1206_3216Metric_Pad1.30x1.75mm_HandSolder, F.Cu at (119.9, 77.5)
- added TP1: Cartridge reset (cart slot B2), TestPoint:TestPoint_Loop_D2.54mm_Drill1.5mm_Beaded, F.Cu at (263.7, 66.9)
- added TP10: Extra address A_{20}, TestPoint:TestPoint_Loop_D2.54mm_Drill1.5mm_Beaded, F.Cu at (268.8, 87.1)
- added TP11: Extra address A_{21}, TestPoint:TestPoint_Loop_D2.54mm_Drill1.5mm_Beaded, F.Cu at (273.8, 66.9)
- added TP12: Extra address A_{22}, TestPoint:TestPoint_Loop_D2.54mm_Drill1.5mm_Beaded, F.Cu at (273.8, 71.9)
- added TP13: Extra address A_{23}, TestPoint:TestPoint_Loop_D2.54mm_Drill1.5mm_Beaded, F.Cu at (273.8, 77.0)
- added TP2: Cartridge chip enable (cart slot B17), TestPoint:TestPoint_Loop_D2.54mm_Drill1.5mm_Beaded, F.Cu at (263.7, 71.9)
- added TP3: Cartridge address strobe (cart slot B18), TestPoint:TestPoint_Loop_D2.54mm_Drill1.5mm_Beaded, F.Cu at (263.7, 77.0)
- added TP4: Cartridge 68K data clock (cart slot B19), TestPoint:TestPoint_Loop_D2.54mm_Drill1.5mm_Beaded, F.Cu at (263.7, 82.0)
- added TP5: Cartridge data xfer ack (cart slot B20), TestPoint:TestPoint_Loop_D2.54mm_Drill1.5mm_Beaded, F.Cu at (263.7, 87.1)
- added TP6: Cartridge ??? signal (cart slot B31), TestPoint:TestPoint_Loop_D2.54mm_Drill1.5mm_Beaded, F.Cu at (268.8, 66.9)
- added TP7: Unused expansion port signal, TestPoint:TestPoint_Loop_D2.54mm_Drill1.5mm_Beaded, F.Cu at (268.8, 71.9)
- added TP8: Extra address A_{18}, TestPoint:TestPoint_Loop_D2.54mm_Drill1.5mm_Beaded, F.Cu at (268.8, 77.0)
- added TP9: Extra address A_{19}, TestPoint:TestPoint_Loop_D2.54mm_Drill1.5mm_Beaded, F.Cu at (268.8, 82.0)
- J1: value Mega CD Header -> Address_Connector; footprint Sega:PinHeader_2x30_P2.54mm_Vertical_AB_Numbering -> Sega:PinHeader_2x20_P2.54mm_Vertical_LeftRight_Numbering
- J2: value Tera Drive Expansion Port -> Data_Control_Connector; footprint Sega:TE_1761469-1_BA_Numbering -> Sega:PinHeader_2x30_P2.54mm_Vertical_LeftRight_Numbering; moved to F.Cu
- R1: footprint Resistor_THT:R_Axial_DIN0207_L6.3mm_D2.5mm_P10.16mm_Horizontal -> Resistor_SMD:R_1206_3216Metric_Pad1.30x1.75mm_HandSolder
- R2: value 300Ω -> 100Ω; footprint Resistor_THT:R_Axial_DIN0207_L6.3mm_D2.5mm_P10.16mm_Horizontal -> Resistor_SMD:R_1206_3216Metric_Pad1.30x1.75mm_HandSolder
- moved J1 74.2 mm to (89.4, 72.6), turned to 90 degrees
- moved J2 46.1 mm to (63.0, 59.9)
- moved R1 40.7 mm to (89.4, 77.7)
- moved REF** 22.9 mm to (78.8, 146.1)
- moved R2 19.4 mm to (94.5, 77.7), turned to 90 degrees
- moved REF** 11.3 mm to (69.5, 146.2)
Connections:
- R1 pad 1: Net-(D1-K) -> A_{1}
- R1 pad 2: GND -> VA_{1}
- R2 pad 1: Net-(D2-K) -> A_{2}
- R2 pad 2: GND -> VA_{2}
Routing:
- net GND: track 590.8 -> 0.00 mm, vias 65 -> 0
- net VCC: track 264.8 -> 0.00 mm
- net A_{17}: track 159.1 -> 0.00 mm, vias 1 -> 0
- net D_{2}: track 151.8 -> 0.00 mm, vias 4 -> 0
- net A_{16}: track 150.5 -> 0.00 mm, vias 1 -> 0
- net D_{1}: track 132.9 -> 0.00 mm, vias 4 -> 0
- net D_{5}: track 132.4 -> 0.00 mm, vias 2 -> 0
- net +9V: track 127.2 -> 0.00 mm
- net D_{4}: track 115.9 -> 0.00 mm, vias 4 -> 0
- net A_{13}: track 114.6 -> 0.00 mm, vias 2 -> 0
- net D_{3}: track 114.6 -> 0.00 mm, vias 4 -> 0
- net A_{18}: track 105.2 -> 0.00 mm, vias 2 -> 0
- net A_{11}: track 102.2 -> 0.00 mm, vias 1 -> 0
- net ~{RAS2}: track 98.6 -> 0.00 mm, vias 2 -> 0
- net A_{7}: track 92.9 -> 0.00 mm, vias 1 -> 0
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- removed copper zone on B.Cu, net GND
- removed copper zone on F.Cu, net GND
Other:
- board size 63.8 x 87.4 mm -> 80.9 x 95.2 mm
- board text removed: "+5V"
- board text removed: "+9V"
- board text removed: "A1"
- board text removed: "A30"
- board text removed: "B1"
- board text removed: "B30"
- board text removed: "LEFT"
- board text removed: "RIGHT"
- board text removed: "SOUND1"
- board text removed: "SOUND2"
- board text removed: "SOUND3"
- board text removed: "UNUSED"
- board text removed: "WayWayWay"
