File: Teradrive Mega CD Adapter.kicad_sch (KiCad schematic)
At the start: 75 parts, among them J1 Mega CD Header, J2 Tera Drive Expansion Port

Commit message: Work on v2
Parts:
- removed C1: 47μF, Capacitor_THT:CP_Radial_D5.0mm_P2.50mm, symbol Device:C_Polarized_US
- removed C2: 47μF, Capacitor_THT:CP_Radial_D5.0mm_P2.50mm, symbol Device:C_Polarized
- removed D1: +5V Indicator, LED_THT:LED_D3.0mm, symbol Device:LED
- removed D2: +9V Indicator, LED_THT:LED_D3.0mm, symbol Device:LED
- removed J1: Mega CD Header, Sega:PinHeader_2x30_P2.54mm_Vertical_AB_Numbering, symbol Sega:Conn_02x30_Row_Letter_First_Capitalized
- removed JPA1, JPA11, JPA12, JPA13, JPA14, JPA15, JPA16, JPA17, JPA22, JPA23, JPA24, JPA25, JPA26, JPA27, JPA28, JPA29, JPA3, JPA32, JPA4, JPA5, JPA6, JPB1, JPB10, JPB11, JPB12, JPB13, JPB14, JPB15, JPB16, JPB17, JPB18, JPB19, JPB20, JPB21, JPB22, JPB23, JPB24, JPB25, JPB26, JPB27, JPB28, JPB29, JPB3, JPB30, JPB32, JPB4, JPB5, JPB6, JPB7, JPB8, JPB9: SolderJumper_2_Open, Sega:SolderJumper-2_P1.3mm_Open_RoundedPad1.0x1.5mm_PretendShorted, symbol Sega:SolderJumper_2_Open_PretendClosed
- removed JPB2: Sound 1 Left/Right, Connector_PinHeader_2.54mm:PinHeader_1x03_P2.54mm_Vertical, symbol Jumper:Jumper_3_Open
- removed JPB31: Sound 2 Left/Right, Connector_PinHeader_2.54mm:PinHeader_1x03_P2.54mm_Vertical, symbol Jumper:Jumper_3_Open
- removed TP9V1: MegaCD +9V, TestPoint:TestPoint_Pad_D1.5mm, symbol Connector:TestPoint
- removed TPSL3: MegaCD Sound Left 3 (unused), TestPoint:TestPoint_Pad_D1.5mm, symbol Connector:TestPoint
- removed TPSR3: MegaCD Sound Right 3 (unused), TestPoint:TestPoint_Pad_D1.5mm, symbol Connector:TestPoint
- added J1: Address_Connector, Connector_PinHeader_2.54mm:PinHeader_2x20_P2.54mm_Vertical, symbol Sega:Address_Connector
- added J2: Data_Control_Connector, Connector_PinHeader_2.54mm:PinHeader_2x30_P2.54mm_Vertical, symbol Sega:Data_Control_Connector
- added R10, R11, R12, R13, R14, R15, R16, R17, R18, R19, R20, R21, R22, R23, R24, R25, R26, R27, R28, R29, R30, R31, R32, R33, R34, R35, R36, R37, R38, R39, R40, R41, R42, R43, R44, R45, R46, R5, R6, R7, R8, R9: 100Ω, Resistor_SMD:R_1206_3216Metric_Pad1.30x1.75mm_HandSolder, symbol Device:R_US
- added TP7: Unused expansion port signal, TestPoint:TestPoint_Loop_D2.54mm_Drill1.5mm_Beaded, symbol Connector:TestPoint
- added TP8: Extra address A_{18}, TestPoint:TestPoint_Loop_D2.54mm_Drill1.5mm_Beaded, symbol Connector:TestPoint
- added TP9: Extra address A_{19}, TestPoint:TestPoint_Loop_D2.54mm_Drill1.5mm_Beaded, symbol Connector:TestPoint
- R1: footprint Resistor_THT:R_Axial_DIN0207_L6.3mm_D2.5mm_P10.16mm_Horizontal -> Resistor_SMD:R_1206_3216Metric_Pad1.30x1.75mm_HandSolder
- R2: value 300Ω -> 100Ω; footprint Resistor_THT:R_Axial_DIN0207_L6.3mm_D2.5mm_P10.16mm_Horizontal -> Resistor_SMD:R_1206_3216Metric_Pad1.30x1.75mm_HandSolder
- TP1: renamed from TPA2; value Tera Drive cartridge reset (cart slot B2) -> Cartridge reset (cart slot B2); footprint TestPoint:TestPoint_Pad_D1.5mm -> TestPoint:TestPoint_Loop_D2.54mm_Drill1.5mm_Beaded
- TP10: renamed from TPA7; value Tera Drive extra address A_{20} -> Extra address A_{20}; footprint TestPoint:TestPoint_Pad_D1.5mm -> TestPoint:TestPoint_Loop_D2.54mm_Drill1.5mm_Beaded
- TP11: renamed from TPA8; value Tera Drive extra address A_{21} -> Extra address A_{21}; footprint TestPoint:TestPoint_Pad_D1.5mm -> TestPoint:TestPoint_Loop_D2.54mm_Drill1.5mm_Beaded
- TP12: renamed from TPA9; value Tera Drive extra address A_{22} -> Extra address A_{22}; footprint TestPoint:TestPoint_Pad_D1.5mm -> TestPoint:TestPoint_Loop_D2.54mm_Drill1.5mm_Beaded
- TP13: renamed from TPA10; value Tera Drive extra address A_{23} -> Extra address A_{23}; footprint TestPoint:TestPoint_Pad_D1.5mm -> TestPoint:TestPoint_Loop_D2.54mm_Drill1.5mm_Beaded
- TP2: renamed from TPA18; value Tera Drive cartridge chip enable (cart slot B17) -> Cartridge chip enable (cart slot B17); footprint TestPoint:TestPoint_Pad_D1.5mm -> TestPoint:TestPoint_Loop_D2.54mm_Drill1.5mm_Beaded
- TP3: renamed from TPA19; value Tera Drive cartridge address strobe (cart slot B18) -> Cartridge address strobe (cart slot B18); footprint TestPoint:TestPoint_Pad_D1.5mm -> TestPoint:TestPoint_Loop_D2.54mm_Drill1.5mm_Beaded
- TP4: renamed from TPA20; value Tera Drive cartridge 68K data clock (cart slot B19) -> Cartridge 68K data clock (cart slot B19); footprint TestPoint:TestPoint_Pad_D1.5mm -> TestPoint:TestPoint_Loop_D2.54mm_Drill1.5mm_Beaded
- TP5: renamed from TPA21; value Tera Drive cartridge data xfer ack (cart slot B20) -> Cartridge data xfer ack (cart slot B20); footprint TestPoint:TestPoint_Pad_D1.5mm -> TestPoint:TestPoint_Loop_D2.54mm_Drill1.5mm_Beaded
- TP6: renamed from TPA30; value Tera Drive cartridge ??? signal (cart slot B31) -> Cartridge ??? signal (cart slot B31); footprint TestPoint:TestPoint_Pad_D1.5mm -> TestPoint:TestPoint_Loop_D2.54mm_Drill1.5mm_Beaded
- renumbered J2 to J5, JPA31 to JP1
Connections:
- net SOUND1 is gone; now on net SL2: J5.B2 (Pin_b2)
- net SOUND2 is gone; now on net SR2: J5.B31 (Pin_b31)
- net ~{DISK} is gone; now on net GND: J5.A15 (Pin_a15)
- net +5V: now also J1.19 (VCC), J1.20 (VCC)
- net A_{10}: now also R12.1
- net A_{11}: now also R13.1
- net A_{12}: now also R14.1
- net A_{13}: now also R15.1
- net A_{14}: now also R16.1
- net A_{15}: now also R17.1
- net A_{16}: now also R18.1
- net A_{17}: now also R19.1
- net A_{18}: now also TP8.1
- net A_{19}: now also TP9.1
- net A_{1}: now also R1.1
- net A_{2}: now also R2.1
- net A_{3}: now also R5.1
- net A_{4}: now also R6.1
- net A_{5}: now also R7.1
- net A_{6}: now also R8.1
- net A_{7}: now also R9.1
- net A_{8}: now also R10.1
- net A_{9}: now also R11.1
- net D_{0}: now also R22.1
- net D_{10}: now also R32.1
- net D_{11}: now also R33.1
- net D_{12}: now also R34.1
- net D_{13}: now also R35.1
- net D_{14}: now also R36.1
- net D_{15}: now also R37.1
- net D_{1}: now also R23.1
- net D_{2}: now also R24.1
- net D_{3}: now also R25.1
- net D_{4}: now also R26.1
- net D_{5}: now also R27.1
- net D_{6}: now also R28.1
- net D_{7}: now also R29.1
- net D_{8}: now also R30.1
- net D_{9}: now also R31.1
- net FRES: now also R46.1
- net GND: now also J1.18 (GND), J1.21 (GND), J1.22 (GND), J1.23 (GND), J1.24 (GND), J1.25 (GND), J1.26 (GND), J1.27 (GND), J1.28 (GND), J1.29 (GND), J1.30 (GND), J1.31 (GND), J1.32 (GND), J1.33 (GND), J1.34 (GND), J1.35 (GND), J1.36 (GND), J1.37 (GND), J1.38 (GND), J1.39 (GND), J1.40 (GND), J2.17 (GND), J2.31 (GND), J2.32 (GND), J2.33 (GND), J2.34 (GND), J2.35 (GND), J2.36 (GND), J2.37 (GND), J2.38 (GND), J2.39 (GND), J2.40 (GND), J2.41 (GND), J2.42 (GND), J2.43 (GND), J2.44 (GND), J2.45 (GND), J2.46 (GND), J2.47 (GND), J2.48 (GND), J2.49 (GND), J2.50 (GND), J2.51 (GND), J2.52 (GND), J2.53 (GND), J2.54 (GND), J2.55 (GND), J2.56 (GND); no longer R1.2, R2.2
- net SL2: now also J2.28 (SL2), R20.1
- net SR2: now also J2.30 (SR2), R21.1
- net ~{ASEL}: now also R41.1
- net ~{CAS0}: now also R38.1
- net ~{CAS2}: now also R39.1
- net ~{FDC}: now also R45.1
- net ~{FDWR}: now also TP7.1
- net ~{LWR}: now also R42.1
- net ~{RAS2}: now also R44.1
- net ~{ROM}: now also R43.1
- net ~{UWR}: now also R40.1
- new net GNDA: J2.27 (AGND), J2.29 (AGND), J2.57 (AGND), J2.58 (AGND), J2.59 (AGND), J2.60 (AGND), R20.2, R21.2
- new net VA_{10}: J1.16 (VA_{10}), R12.2
- new net VA_{11}: J1.14 (VA_{11}), R13.2
- new net VA_{12}: J1.12 (VA_{12}), R14.2
- new net VA_{13}: J1.10 (VA_{13}), R15.2
- new net VA_{14}: J1.8 (VA_{14}), R16.2
- new net VA_{15}: J1.6 (VA_{15}), R17.2
- new net VA_{16}: J1.4 (VA_{16}), R18.2
- new net VA_{17}: J1.2 (VA_{17}), R19.2
- new net VA_{1}: J1.1 (VA_{1}), R1.2
- new net VA_{2}: J1.3 (VA_{2}), R2.2
- new net VA_{3}: J1.5 (VA_{3}), R5.2
- new net VA_{4}: J1.7 (VA_{4}), R6.2
- new net VA_{5}: J1.9 (VA_{5}), R7.2
- new net VA_{6}: J1.11 (VA_{6}), R8.2
- new net VA_{7}: J1.13 (VA_{7}), R9.2
- new net VA_{8}: J1.15 (VA_{8}), R10.2
- new net VA_{9}: J1.17 (VA_{9}), R11.2
- new net VD_{0}: J2.1 (VD_{0}), R22.2
- new net VD_{10}: J2.12 (VD_{10}), R32.2
- new net VD_{11}: J2.10 (VD_{11}), R33.2
- new net VD_{12}: J2.8 (VD_{12}), R34.2
- new net VD_{13}: J2.6 (VD_{13}), R35.2
- new net VD_{14}: J2.4 (VD_{14}), R36.2
- new net VD_{15}: J2.2 (VD_{15}), R37.2
- new net VD_{1}: J2.3 (VD_{1}), R23.2
- new net VD_{2}: J2.5 (VD_{2}), R24.2
- new net VD_{3}: J2.7 (VD_{3}), R25.2
- new net VD_{4}: J2.9 (VD_{4}), R26.2
- new net VD_{5}: J2.11 (VD_{5}), R27.2
- new net VD_{6}: J2.13 (VD_{6}), R28.2
- new net VD_{7}: J2.15 (VD_{7}), R29.2
- new net VD_{8}: J2.16 (VD_{8}), R30.2
- new net VD_{9}: J2.14 (VD_{9}), R31.2
- new net VFRES: J2.18 (~{VFRES}), R46.2
- new net ~{VASEL}: J2.21 (~{VASEL}), R41.2
- new net ~{VCAS0}: J2.19 (~{VCAS0}), R38.2
- new net ~{VCAS2}: J2.23 (~{VCAS2}), R39.2
- new net ~{VFDC}: J2.24 (~{VFDC}), R45.2
- new net ~{VLWR}: J2.26 (~{VLWR}), R42.2
- new net ~{VRAS2}: J2.25 (~{VRAS2}), R44.2
- new net ~{VROM}: J2.22 (~{VROM}), R43.2
- new net ~{VUWR}: J2.20 (~{VUWR}), R40.2
Other:
- note added: "Address Terminators"
- note added: "Audio Terminators"
- note added: "Control Terminators"
- note added: "Data Terminators"
- note added: "Unused pins"
- note removed: "*1"
- note removed: "*1 +9V (+7V min) comes from Mega Drive/Tera Drive to act as a power switch for the Mega CD. See link."
- note removed: "*1 It is currently unknown which sound pin is left or right"
- note removed: "*2"
- note removed: "*2 ~{DISK} immediately connects to ground inside the Mega CD"
- note removed: "1"
- note removed: "10"
- note removed: "20"
- note removed: "30"
- note removed: "32"
- note removed: "A"
- note removed: "B"
- note removed: "Blinkenlights"
- note removed: "MegaCD Connector Extra Pins"
- note removed: "NC"
- note removed: "Tera Drive Connector Duplicate Cartridge Pins"
- note removed: "Tera Drive Connector Extra Address Lines"
- note removed: "Tera Drive Expansion Port Breakout"
- moved on the sheet: JP1, TP1, TP10, TP11, TP12, TP13, TP2, TP3, TP4, TP5, TP6
